File: hardware/gpx_extend.sch (EAGLE design)
At the start: 22 parts, among them SW1 SW-SPST, U1 STM32L011F4PX

Commit message: fix DMA transfer bug at lower baudrates
Parts:
- added D2: UCLAMP3301HSOD523, misc:UCLAMP3301HSOD523
- added R5, R6: 220, misc:R-EU-0603
- C1, C2, C3, C4, C5, C6, C7: device misc:C0603-S -> misc:C-EU-0603
- R1, R2, R3, R4: device misc:R0603-S -> misc:R-EU-0603
Connections:
- new net N$1: D2.C, R6.1, RJ11.5
- new net RX: R5.2, U1.PA10
- net D_IO: now also R5.1, R6.2; no longer RJ11.5, U1.PA10
- net GND: now also D2.A
Other:
- moved on the sheet: RJ11
Changed lines of the file:
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@@
 <part name="P+3" library="supply1" library_urn="urn:adsk.eagle:library:371" deviceset="+5V" device=""/>
 <part name="GND7" library="supply1" library_urn="urn:adsk.eagle:library:371" deviceset="GND" device=""/>
-<part name="C2" library="misc" deviceset="C0603-S" device="" value="4u7"/>
-<part name="C4" library="misc" deviceset="C0603-S" device="" value="100n"/>
-<part name="C3" library="misc" deviceset="C0603-S" device="" value="100n"/>
-<part name="C1" library="misc" deviceset="C0603-S" device="" value="4u7"/>
-<part name="C5" library="misc" deviceset="C0603-S" device="" value="100n"/>
+<part name="C2" library="misc" deviceset="C-EU" device="-0603" value="4u7"/>
+<part name="C4" library="misc" deviceset="C-EU" device="-0603" value="100n"/>
+<part name="C3" library="misc" deviceset="C-EU" device="-0603" value="100n"/>
+<part name="C1" library="misc" deviceset="C-EU" device="-0603" value="4u7"/>
+<part name="C5" library="misc" deviceset="C-EU" device="-0603" value="100n"/>
 <part name="GND8" library="supply1" library_urn="urn:adsk.eagle:library:371" deviceset="GND" device=""/>
-<part name="R1" library="misc" deviceset="R0603-S" device="" value="10k"/>
+<part name="R1" library="misc" deviceset="R-EU" device="-0603" value="10k"/>
 <part name="GND9" library="supply1" library_urn="urn:adsk.eagle:library:371" deviceset="GND" device=""/>
 <part name="+3V4" library="supply1" library_urn="urn:adsk.eagle:library:371" deviceset="+3V3" device=""/>
-<part name="C6" library="misc" deviceset="C0603-S" device="" value="1u"/>
-<part name="C7" library="misc" deviceset="C0603-S" device="" value="4u7"/>
-<part name="R4" library="misc" deviceset="R0603-S" device="" value="1k"/>
-<part name="R3" library="misc" deviceset="R0603-S" device="" value="220"/>
+<part name="C6" library="misc" deviceset="C-EU" device="-0603" value="1u"/>
+<part name="C7" library="misc" deviceset="C-EU" device="-0603" value="4u7"/>
+<part name="R4" library="misc" deviceset="R-EU" device="-0603" value="1k"/>
+<part name="R3" library="misc" deviceset="R-EU" device="-0603" value="220"/>
 <part name="+3V5" library="supply1" library_urn="urn:adsk.eagle:library:371" deviceset="+3V3" device=""/>
 <part name="D1" library="misc" deviceset="LED-DUAL" device=""/>
@@
 <part name="C" library="testpad" library_urn="urn:adsk.eagle:library:385" deviceset="TP" device="TP10R" package3d_urn="urn:adsk.eagle:package:27959/1"/>
 <part name="R" library="testpad" library_urn="urn:adsk.eagle:library:385" deviceset="TP" device="TP10R" package3d_urn="urn:adsk.eagle:package:27959/1"/>
-<part name="R2" library="misc" deviceset="R0603-S" device="" value="2.2k"/>
+<part name="R2" library="misc" deviceset="R-EU" device="-0603" value="2.2k"/>
 <part name="GOLD_ORB_SM1" library="oshw" deviceset="OSHWLOGO" device="LOGO5MM"/>
 <part name="U$1" library="misc" deviceset="GPX_LOGO" device=""/>
+<part name="R5" library="misc" deviceset="R-EU" device="-0603" value="220"/>
+<part name="D2" library="misc" deviceset="UCLAMP3301H" device="SOD523"/>
+<part name="GND1" library="supply1" library_urn="urn:adsk.eagle:library:371" deviceset="GND" device=""/>
+<part name="R6" library="misc" deviceset="R-EU" device="-0603" value="220"/>
 </parts>
 <sheets>
@@
 <instances>
 <instance part="U1" gate="G$1" x="68.58" y="66.04"/>
-<instance part="RJ11" gate="G$1" x="124.46" y="93.98" rot="MR90"/>
-<instance part="P+2" gate="1" x="139.7" y="96.52" rot="MR0"/>
-<instance part="GND3" gate="1" x="116.84" y="86.36" rot="MR0"/>
-<instance part="GND4" gate="1" x="124.46" y="86.36" rot="MR0"/>
+<instance part="RJ11" gate="G$1" x="132.08" y="93.98" rot="MR90"/>
+<instance part="P+2" gate="1" x="147.32" y="96.52" rot="MR0"/>
+<instance part="GND3" gate="1" x="124.46" y="86.36" rot="MR0"/>
+<instance part="GND4" gate="1" x="132.08" y="86.36" rot="MR0"/>
 <instance part="NRF" gate="A" x="91.44" y="119.38"/>
-<instance part="GND5" gate="1" x="68.58" y="129.54" rot="MR0"/>
+<instance part="GND5" gate="1" x="78.74" y="129.54" rot="MR0"/>
 <instance part="+3V1" gate="G$1" x="101.6" y="134.62"/>
 <instance part="+3V2" gate="G$1" x="91.44" y="71.12" rot="MR0"/>
@@
 <instance part="GOLD_ORB_SM1" gate="G$1" x="-38.1" y="78.74"/>
 <instance part="U$1" gate="G$1" x="-25.4" y="63.5"/>
+<instance part="R5" gate="G$1" x="96.52" y="78.74" rot="R180"/>
+<instance part="D2" gate="G$1" x="127" y="68.58" rot="R90"/>
+<instance part="GND1" gate="1" x="127" y="60.96" rot="MR0"/>
+<instance part="R6" gate="G$1" x="119.38" y="73.66" rot="R180"/>
 </instances>
 <busses>
@@
 <segment>
 <pinref part="RJ11" gate="G$1" pin="1"/>
-<wire x1="129.54" y1="91.44" x2="129.54" y2="86.36" width="0.1524" layer="91"/>
+<wire x1="137.16" y1="91.44" x2="137.16" y2="86.36" width="0.1524" layer="91"/>
 <pinref part="P+2" gate="1" pin="+5V"/>
-<wire x1="139.7" y1="86.36" x2="139.7" y2="93.98" width="0.1524" layer="91"/>
-<wire x1="139.7" y1="86.36" x2="129.54" y2="86.36" width="0.1524" layer="91"/>
+<wire x1="147.32" y1="86.36" x2="147.32" y2="93.98" width="0.1524" layer="91"/>
+<wire x1="147.32" y1="86.36" x2="137.16" y2="86.36" width="0.1524" layer="91"/>
 <pinref part="RJ11" gate="G$1" pin="2"/>
-<wire x1="127" y1="91.44" x2="127" y2="86.36" width="0.1524" layer="91"/>
-<wire x1="127" y1="86.36" x2="129.54" y2="86.36" width="0.1524" layer="91"/>
-<junction x="129.54" y="86.36"/>
+<wire x1="134.62" y1="91.44" x2="134.62" y2="86.36" width="0.1524" layer="91"/>
+<wire x1="134.62" y1="86.36" x2="137.16" y2="86.36" width="0.1524" layer="91"/>
+<junction x="137.16" y="86.36"/>
 </segment>
 <segment>
@@
 <pinref part="U2" gate="G$1" pin="EN"/>
 <wire x1="-22.86" y1="121.92" x2="-22.86" y2="127" width="0.1524" layer="91"/>
+<junction x="-22.86" y="127"/>
 </segment>
 </net>
@@
 <pinref part="RJ11" gate="G$1" pin="6"/>
 <pinref part="GND3" gate="1" pin="GND"/>
-<wire x1="116.84" y1="91.44" x2="116.84" y2="88.9" width="0.1524" layer="91"/>
+<wire x1="124.46" y1="91.44" x2="124.46" y2="88.9" width="0.1524" layer="91"/>
 </segment>
 <segment>
 <pinref part="RJ11" gate="G$1" pin="3"/>
 <pinref part="GND4" gate="1" pin="GND"/>
-<wire x1="124.46" y1="88.9" x2="124.46" y2="91.44" width="0.1524" layer="91"/>
+<wire x1="132.08" y1="88.9" x2="132.08" y2="91.44" width="0.1524" layer="91"/>
 </segment>
 <segment>
@@
 <wire x1="88.9" y1="124.46" x2="83.82" y2="124.46" width="0.1524" layer="91"/>
 <wire x1="83.82" y1="124.46" x2="83.82" y2="132.08" width="0.1524" layer="91"/>
-<wire x1="83.82" y1="132.08" x2="68.58" y2="132.08" width="0.1524" layer="91"/>
+<wire x1="83.82" y1="132.08" x2="78.74" y2="132.08" width="0.1524" layer="91"/>
 <pinref part="GND5" gate="1" pin="GND"/>
 </segment>
@@
 <wire x1="25.4" y1="88.9" x2="25.4" y2="86.36" width="0.1524" layer="91"/>
 </segment>
+<segment>
+<pinref part="D2" gate="G$1" pin="A"/>
+<pinref part="GND1" gate="1" pin="GND"/>
+<wire x1="127" y1="63.5" x2="127" y2="66.04" width="0.1524" layer="91"/>
+</segment>
 </net>
 <net name="D_IO" class="0">
 <segment>
-<pinref part="RJ11" gate="G$1" pin="5"/>
-<wire x1="119.38" y1="91.44" x2="119.38" y2="73.66" width="0.1524" layer="91"/>
 <pinref part="U1" gate="G$1" pin="PA9"/>
-<pinref part="U1" gate="G$1" pin="PA10"/>
-<wire x1="91.44" y1="78.74" x2="88.9" y2="78.74" width="0.1524" layer="91"/>
-<wire x1="91.44" y1="78.74" x2="91.44" y2="73.66" width="0.1524" layer="91"/>
-<wire x1="91.44" y1="73.66" x2="88.9" y2="73.66" width="0.1524" layer="91"/>
-<label x="91.44" y="78.74" size="1.778" layer="95" rot="MR180" xref="yes"/>
-<wire x1="91.44" y1="73.66" x2="119.38" y2="73.66" width="0.1524" layer="91"/>
+<wire x1="88.9" y1="73.66" x2="104.14" y2="73.66" width="0.1524" layer="91"/>
+<pinref part="R5" gate="G$1" pin="1"/>
+<wire x1="101.6" y1="78.74" x2="104.14" y2="78.74" width="0.1524" layer="91"/>
+<wire x1="104.14" y1="78.74" x2="104.14" y2="73.66" width="0.1524" layer="91"/>
+<label x="104.14" y="78.74" size="1.778" layer="95" xref="yes"/>
+<pinref part="R6" gate="G$1" pin="2"/>
+<wire x1="114.3" y1="73.66" x2="104.14" y2="73.66" width="0.1524" layer="91"/>
+<junction x="104.14" y="73.66"/>
 </segment>
 <segment>
@@
 </segment>
 </net>
+<net name="RX" class="0">
+<segment>
+<pinref part="U1" gate="G$1" pin="PA10"/>
+<pinref part="R5" gate="G$1" pin="2"/>
+<wire x1="91.44" y1="78.74" x2="88.9" y2="78.74" width="0.1524" layer="91"/>
+</segment>
+</net>
+<net name="N$1" class="0">
+<segment>
+<pinref part="RJ11" gate="G$1" pin="5"/>
+<wire x1="127" y1="91.44" x2="127" y2="73.66" width="0.1524" layer="91"/>
+<pinref part="R6" gate="G$1" pin="1"/>
+<pinref part="D2" gate="G$1" pin="C"/>
+<wire x1="127" y1="71.12" x2="127" y2="73.66" width="0.1524" layer="91"/>
+<wire x1="127" y1="73.66" x2="124.46" y2="73.66" width="0.1524" layer="91"/>
+<junction x="127" y="73.66"/>
+</segment>
+</net>
